File: KiCad/RobocupSwinderPCB/RobocupSwinderPCB.kicad_sch (KiCad schematic)
At the start: 19 parts, among them J1 Barrel_Jack, M1 Stepper_Motor_bipolar, M2 Stepper_Motor_bipolar, SW2 SW_DPDT_x2, SW3 SW_SPST, U1 Teensy4.1, U2 TSR_1-2450

Commit message: Updated pin assignments.
Parts:
- removed 1: ~, symbol Library:WC1602_Display_(4_Pins)
- added LCD1: ~, Connector_JST:JST_XH_B4B-XH-A_1x04_P2.50mm_Vertical, symbol Library:WC1602_Display_(4_Pins)
- added R1, R2: 10K, Resistor_SMD:R_1206_3216Metric_Pad1.30x1.75mm_HandSolder, symbol Device:R
- added R3, R4: 1K, Resistor_SMD:R_1206_3216Metric_Pad1.30x1.75mm_HandSolder, symbol Device:R
- added SW1: Limit_Switch, Connector_JST:JST_XH_B3B-XH-A_1x03_P2.50mm_Vertical, symbol Switch:SW_DPDT_x2
- A1: value Pololu_Breakout_DRV8825 -> DRV8825_Feed
- A2: value Pololu_Breakout_DRV8825 -> DRV8825_Coil
- C1, C2: value C_Polarized -> 100uF; footprint (none) -> Capacitor_THT:CP_Radial_D8.0mm_P3.50mm
- C3, C4: value C -> 10uF; footprint (none) -> Capacitor_SMD:C_1206_3216Metric_Pad1.33x1.80mm_HandSolder
- D1, D2: footprint (none) -> LED_SMD:LED_1206_3216Metric_Pad1.42x1.75mm_HandSolder
- F1: value Fuse -> 4.5A; footprint (none) -> Fuse:Fuse_1206_3216Metric
- L1: value L -> 5.6uH; footprint (none) -> Inductor_SMD:L_TracoPower_TCK-141
- M1, M2: footprint (none) -> Connector_JST:JST_XH_B4B-XH-A_1x04_P2.50mm_Vertical
- RE1: footprint (none) -> Connector_JST:JST_XH_B5B-XH-A_1x05_P2.50mm_Vertical
- SW2: value SW_DPDT_x2 -> Limit_Switch; footprint (none) -> Connector_JST:JST_XH_B3B-XH-A_1x03_P2.50mm_Vertical
- SW3: footprint (none) -> Connector_JST:JST_XH_B2B-XH-A_1x02_P2.50mm_Vertical
- U1: footprint (none) -> TeensyLibrary:Teensy4.1 Pins-only
Connections:
- net +3.3V: now also RE1.2 (VCC), R1.1, R2.1
- net +5V: now also A1.10 (M0), A1.13 (~{RST}), A2.13 (~{RST}), D2.2 (A), LCD1.2 (VCC)
- net GND: now also A1.1 (GND), A1.11 (M1), A1.12 (M2), A1.7 (GND), A2.1 (GND), A2.10 (M0), A2.11 (M1), A2.12 (M2), A2.7 (GND), J1.2, RE1.1 (GND), SW2.1 (A), LCD1.1 (GND), R3.2, R4.2, SW1.1 (A); no longer J1.1
- net VCC: now also C1.1, C2.1, D1.2 (A)
- net at U1.40 (18_A4_SDA): now also LCD1.4 (SDA)
- net at U1.41 (19_A5_SCL): now also LCD1.3 (SCL)
- net at RE1.3 (CLK): now also U1.43 (21_A7_RX5_BCLK1)
- net at RE1.4 (DT): now also U1.44 (22_A8_CTX1)
- net at RE1.5 (SW): now also U1.45 (23_A9_CRX1_MCLK1)
- net at U1.21 (29_TX7): now also A2.2 (~{FLT})
- net at U1.22 (30_CRX3): now also A1.2 (~{FLT})
- net at U1.27 (35_TX8): now also A2.14 (~{SLP})
- net at U1.28 (36_CS): now also A2.15 (STEP)
- net at U1.29 (37_CS): now also A2.16 (DIR)
- net at U1.30 (38_CS1_IN1): now also A1.15 (STEP)
- net at U1.31 (39_MISO1_OUT1A): now also A1.16 (DIR)
- net at U1.32 (40_A16): now also A1.14 (~{SLP})
- net at U1.7 (5_IN2): now also SW1.2 (B)
- net at U1.8 (6_OUT1D): now also SW2.2 (B)
- net at SW2.3 (C): now also R2.2
- net at A1.3 (A2): now also M1.2 (-)
- net at A1.4 (A1): now also M1.1
- net at A1.5 (B1): now also M1.3
- net at A1.6 (B2): now also M1.4
- net at A1.8 (VMOT): now also C1.2
- net at SW3.1 (A): now also J1.1; no longer J1.2
- net at M2.1: now also A2.4 (A1)
- net at M2.2 (-): now also A2.3 (A2)
- net at M2.3: now also A2.5 (B1)
- net at M2.4: now also A2.6 (B2)
- net at D2.1 (K): now also R4.1
- net at C2.2: now also A2.8 (VMOT)
- net at D1.1 (K): now also R3.1
- new net: R1.2, SW1.3 (C)
- no-connect marks 0 -> 50
Other:
- company: (none) -> Robojackets
- title: (none) -> Robocup Swinder
- moved on the sheet: C3, C4, F1, J1, L1, SW2A, SW3, U1, U2

Commit message: A whole lotta stuff.
Parts:
- removed U2: TSR_1-2450, Converter_DCDC:Converter_DCDC_TRACO_TSR-1_THT, symbol Regulator_Switching:TSR_1-2450
- added C5: 0.1uF, Capacitor_SMD:C_1206_3216Metric_Pad1.33x1.80mm_HandSolder, symbol Device:C
- added U3: LM7805_TO220, Package_TO_SOT_SMD:SOT-223, symbol Regulator_Linear:LM7805_TO220
- J1: footprint Connector_BarrelJack:BarrelJack_SwitchcraftConxall_RAPC10U_Horizontal -> Library:CONN1x2_PJ-037A_CUD
Connections:
- net +5V: now also C5.1, U3.3 (VO)
- net GND: now also C5.2, U3.2 (GND), U3.4 (GND)
- net VCC: now also U3.1 (VI)
- net Coil_FLT_Pin_21: now reaches A2.2 (~{FLT}), U1.21 (29_TX7)
- net Feed_FLT_Pin_22: now reaches A1.2 (~{FLT}), U1.22 (30_CRX3)
- net Coil_DIR_Pin_35: now reaches U1.27 (35_TX8)
- net Coil_DIR_Pin_35: now also A2.16 (DIR); no longer A2.14 (~{SLP})
- net Coil_STEP_Pin_36: now reaches A2.15 (STEP), U1.28 (36_CS)
- net Coil_SLP_Pin_37: now reaches U1.29 (37_CS)
- net Coil_SLP_Pin_37: now also A2.14 (~{SLP}); no longer A2.16 (DIR)
- net Feed_DIR_Pin_38: now reaches U1.30 (38_CS1_IN1)
- net Feed_DIR_Pin_38: now also A1.16 (DIR); no longer A1.15 (STEP)
- net Feed_STEP_Pin_39: now reaches U1.31 (39_MISO1_OUT1A)
- net Feed_STEP_Pin_39: now also A1.15 (STEP); no longer A1.16 (DIR)
- net Feed_SLP_Pin_40: now reaches A1.14 (~{SLP}), U1.32 (40_A16)
- net LCD_SDA_Pin_18: now reaches LCD1.4 (SDA), U1.40 (18_A4_SDA)
- net LCD_SCL_Pin_19: now reaches LCD1.3 (SCL), U1.41 (19_A5_SCL)
- net RE_SW_Pin_21: now reaches RE1.3 (CLK), U1.43 (21_A7_RX5_BCLK1)
- net RE_DT_Pin_22: now reaches RE1.4 (DT), U1.44 (22_A8_CTX1)
- net RE_CLK_Pin_23: now reaches RE1.5 (SW), U1.45 (23_A9_CRX1_MCLK1)
- net LSStart_Pin_7: now reaches SW1.2 (B), U1.7 (5_IN2)
- net LSEnd_Pin_8: now reaches SW2.2 (B), U1.8 (6_OUT1D)
- net at M2.1: now also A2.3 (A2); no longer A2.4 (A1)
- net at M2.2 (-): now also A2.4 (A1); no longer A2.3 (A2)
- net at M1.1: now also A1.3 (A2); no longer A1.4 (A1)
- net at M1.2 (-): now also A1.4 (A1); no longer A1.3 (A2)
Other:
- moved on the sheet: C3, C4, D1, D2, F1, L1, R3, R4, SW3

Commit message: Updated pcb layout.
Parts:
- added H1, H2, H3, H4: MountingHole_Pad, MountingHole:MountingHole_2.2mm_M2_DIN965_Pad, symbol Mechanical:MountingHole_Pad
- D1, D2: footprint LED_SMD:LED_1206_3216Metric_Pad1.42x1.75mm_HandSolder -> LED_SMD:LED_0603_1608Metric_Pad1.05x0.95mm_HandSolder
- J1: footprint Library:CONN1x2_PJ-037A_CUD -> Library:CUI_PJ-037A
- R3, R4: footprint Resistor_SMD:R_1206_3216Metric_Pad1.30x1.75mm_HandSolder -> Resistor_SMD:R_0603_1608Metric_Pad0.98x0.95mm_HandSolder
- U1: footprint TeensyLibrary:Teensy4.1 Pins-only -> TeensyLibrary:Teensy41-Pins-Only_Silkscreen
Connections:
- net GND: now also SW1.3 (NC), SW2.3 (NC), H1.1, H2.1, H3.1, H4.1; no longer SW1.1 (A), SW2.1 (A)
- net LCD_SCL_Pin_19: now also LCD1.4 (SCL); no longer LCD1.3 (SCL)
- net LCD_SDA_Pin_18: now also LCD1.3 (SDA); no longer LCD1.4 (SDA)
- net LSEnd_Pin_8: now also SW2.1 (C); no longer SW2.2 (B)
- net LSStart_Pin_7: now also SW1.1 (C); no longer SW1.2 (B)
- net NO_LS1: now reaches R1.2
- net NO_LS1: now also SW1.2 (NO); no longer SW1.3 (C)
- net NO_LS2: now reaches R2.2
- net NO_LS2: now also SW2.2 (NO); no longer SW2.3 (C)
Other:
- note added: "Control and I/O"
- note added: "Mounting Holes"
- note added: "Power Indicator"
- note added: "Power Supply"
- moved on the sheet: A1, A2, C1, C2, C3, C4, C5, D1, F1, J1, L1, LCD1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

Commit message: Routing.
Connections:
- net Coil_FLT_Pin_21 renamed Coil_FLT_Pin_22
- net Coil_FLT_Pin_22: now also U1.22 (30_CRX3); no longer U1.21 (29_TX7)
- net Feed_FLT_Pin_22 renamed Feed_FLT_Pin_21
- net Feed_FLT_Pin_21: now also U1.21 (29_TX7); no longer U1.22 (30_CRX3)
Changed lines of the file:
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@@
 		)
 	)
-	(label "Feed_FLT_Pin_22"
+	(label "Feed_FLT_Pin_21"
 		(at 281.94 135.89 0)
 		(fields_autoplaced yes)
@@
 		)
 	)
-	(label "Coil_FLT_Pin_21"
+	(label "Coil_FLT_Pin_22"
 		(at 279.4 186.69 0)
 		(fields_autoplaced yes)
@@
 		)
 	)
-	(label "Coil_FLT_Pin_21"
+	(label "Feed_FLT_Pin_21"
 		(at 166.37 151.13 0)
 		(fields_autoplaced yes)
@@
 		)
 	)
-	(label "Feed_FLT_Pin_22"
+	(label "Coil_FLT_Pin_22"
 		(at 166.37 153.67 0)
 		(fields_autoplaced yes)
