File: KiCad/RobocupSwinderPCB/RobocupSwinderPCB.kicad_pcb (KiCad board)
At the start: 2 copper layers, 92 x 57 mm, 28 parts, among them J1 Barrel_Jack, M1 Stepper_Motor_bipolar, M2 Stepper_Motor_bipolar, SW1 Limit_Switch, SW2 Limit_Switch, SW3 SW_SPST, U1 Teensy4.1, U3 LM7805_TO220

Commit message: Final commit till v1.0
Connections:
- A1 pad 8: Net-(A1-VMOT) -> VCC
- A2 pad 8: Net-(A2-VMOT) -> VCC
- C1 pad 2: Net-(A1-VMOT) -> GND
- C2 pad 2: Net-(A2-VMOT) -> GND
Routing:
- net VCC: track 69.1 -> 82.0 mm
- net Net-(A2-VMOT): track 10.2 -> 0.00 mm
- net Net-(A1-VMOT): track 9.50 -> 0.00 mm
